File: stepper-tester.sch (KiCad schematic (older format))
At the start: 13 parts

Commit message: Kicad update
Parts:
- removed U?: NE555, symbol Timer:NE555
- added U?: NE555P, Package_DIP:DIP-8_W7.62mm, symbol Timer:NE555P
Connections:
- net 5V: now also U?.4 (R), U?.8 (VCC)
- net GND: now also U?.1 (GND)
- net STEP: now also U?.3 (Q)
- net at C?.2, R?.1, R?.2: now also U?.2 (TR), U?.6 (THR)
- net at C?.2: now also U?.5 (CV)
Changed lines of the file:
@@
 Text GLabel 7450 1500 1    50   Input ~ 0
 VMOT
-$Comp
-L Timer:NE555 U?
-U 1 1 5F1F1E78
-P 2650 5450
-F 0 "U?" H 2900 6000 50  0000 C CNN
-F 1 "NE555" H 2900 5900 50  0000 C CNN
-F 2 "" H 2650 5450 50  0001 C CNN
-F 3 "http://www.ti.com/lit/ds/symlink/ne555.pdf" H 2650 5450 50  0001 C CNN
-	1    2650 5450
-	1    0    0    -1
-$EndComp
 Text GLabel 2650 5050 1    50   Input ~ 0
 5V
@@
 Wire Wire Line
 	4500 3150 4650 3150
+$Comp
+L Timer:NE555P U?
+U 1 1 5F2154E9
+P 2650 5450
+F 0 "U?" H 2850 5950 50  0000 C CNN
+F 1 "NE555P" H 2950 5850 50  0000 C CNN
+F 2 "Package_DIP:DIP-8_W7.62mm" H 3300 5050 50  0001 C CNN
+F 3 "http://www.ti.com/lit/ds/symlink/ne555.pdf" H 3500 5050 50  0001 C CNN
+	1    2650 5450
+	1    0    0    -1
+$EndComp
 $EndSCHEMATC

Commit message: Update schematics
Parts:
- removed D?: D_Zener, symbol Device:D_Zener
- removed RV?: R_POT, symbol Device:R_POT
- added C? (x2): 0.1uF, symbol Device:C
- added U?: AMS1117-5.0, Package_TO_SOT_SMD:SOT-223-3_TabPin2, symbol Regulator_Linear:AMS1117-5.0
- J2: renamed from J?; footprint (none) -> Connector_PinHeader_2.54mm:PinHeader_1x04_P2.54mm_Vertical
- R1, R2: renamed from R?; footprint (none) -> Resistor_THT:R_Axial_DIN0207_L6.3mm_D2.5mm_P2.54mm_Vertical
- RV2: renamed from RV?; footprint (none) -> Connector_PinHeader_2.54mm:PinHeader_1x03_P2.54mm_Vertical
- SW1, SW2: renamed from SW?; footprint (none) -> Button_Switch_THT:SW_NKK_GW12LJP
- gave numbers to parts that had none: 5
Connections:
- net 5V: now also C?.1, U?.2 (VO)
- net GND: now also C?.1, C?.2, U?.1 (GND)
- net VMOT: now also C?.2, U?.3 (VI)
Changed lines of the file:
@@
 $EndDescr
 $Comp
-L Driver_Motor:Pololu_Breakout_DRV8825 A?
+L Driver_Motor:Pololu_Breakout_DRV8825 A1
 U 1 1 5F1C4D7C
 P 7450 2250
-F 0 "A?" H 7700 2950 50  0000 C CNN
+F 0 "A1" H 7700 2950 50  0000 C CNN
 F 1 "DRV8825" H 7700 2850 50  0000 C CNN
 F 2 "Module:Pololu_Breakout-16_15.2x20.3mm" H 7650 1450 50  0001 L CNN
@@
 $EndComp
 $Comp
-L Connector:Barrel_Jack J?
+L Connector:Barrel_Jack J1
 U 1 1 5F1CE645
 P 1700 1450
-F 0 "J?" H 1757 1775 50  0000 C CNN
+F 0 "J1" H 1757 1775 50  0000 C CNN
 F 1 "Barrel_Jack" H 1757 1684 50  0000 C CNN
 F 2 "" H 1750 1410 50  0001 C CNN
@@
 $EndComp
 $Comp
-L power:GND #PWR?
+L power:GND #PWR0101
 U 1 1 5F1CF223
 P 2150 1600
-F 0 "#PWR?" H 2150 1350 50  0001 C CNN
+F 0 "#PWR0101" H 2150 1350 50  0001 C CNN
 F 1 "GND" H 2155 1427 50  0000 C CNN
 F 2 "" H 2150 1600 50  0001 C CNN
@@
 VMOT
 $Comp
-L power:GND #PWR?
+L power:GND #PWR0102
 U 1 1 5F1D1224
 P 7500 3150
-F 0 "#PWR?" H 7500 2900 50  0001 C CNN
+F 0 "#PWR0102" H 7500 2900 50  0001 C CNN
 F 1 "GND" H 7505 2977 50  0000 C CNN
 F 2 "" H 7500 3150 50  0001 C CNN
@@
 Connection ~ 7500 3100
 $Comp
-L Connector:Conn_01x04_Male J?
+L Connector:Conn_01x04_Male J2
 U 1 1 5F1CE36B
 P 8300 2400
-F 0 "J?" H 8272 2328 50  0000 R CNN
+F 0 "J2" H 8272 2328 50  0000 R CNN
 F 1 "Conn_01x04_Male" H 8272 2373 50  0001 R CNN
-F 2 "" H 8300 2400 50  0001 C CNN
+F 2 "Connector_PinHeader_2.54mm:PinHeader_1x04_P2.54mm_Vertical" H 8300 2400 50  0001 C CNN
 F 3 "~" H 8300 2400 50  0001 C CNN
 	1    8300 2400
@@
 	7450 1500 7450 1650
 $Comp
-L Device:D_Zener D?
-U 1 1 5F1D37F7
-P 2700 2050
-F 0 "D?" V 2600 1850 50  0000 L CNN
-F 1 "D_Zener" V 2650 1850 50  0001 L CNN
-F 2 "" H 2700 2050 50  0001 C CNN
-F 3 "~" H 2700 2050 50  0001 C CNN
-	1    2700 2050
-	0    1    1    0
-$EndComp
-Wire Wire Line
-	2000 1350 2700 1350
-$Comp
-L Device:R_POT RV?
-U 1 1 5F1D8352
-P 2700 1550
-F 0 "RV?" H 2630 1550 50  0000 R CNN
-F 1 "R_POT" H 2631 1505 50  0001 R CNN
-F 2 "" H 2700 1550 50  0001 C CNN
-F 3 "~" H 2700 1550 50  0001 C CNN
-	1    2700 1550
-	1    0    0    -1
-$EndComp
-Wire Wire Line
-	2700 1400 2700 1350
-Wire Wire Line
-	2700 1700 2700 1750
-Wire Wire Line
-	2850 1550 2900 1550
-Wire Wire Line
-	2900 1550 2900 1750
-Wire Wire Line
-	2900 1750 2700 1750
-Connection ~ 2700 1750
-$Comp
-L power:GND #PWR?
+L power:GND #PWR0103
 U 1 1 5F1D9BA0
-P 2700 2250
-F 0 "#PWR?" H 2700 2000 50  0001 C CNN
-F 1 "GND" H 2705 2077 50  0000 C CNN
-F 2 "" H 2700 2250 50  0001 C CNN
-F 3 "" H 2700 2250 50  0001 C CNN
-	1    2700 2250
-	1    0    0    -1
-$EndComp
-Wire Wire Line
-	2700 2250 2700 2200
+P 3050 1650
+F 0 "#PWR0103" H 3050 1400 50  0001 C CNN
+F 1 "GND" H 3055 1477 50  0000 C CNN
+F 2 "" H 3050 1650 50  0001 C CNN
+F 3 "" H 3050 1650 50  0001 C CNN
+	1    3050 1650
+	1    0    0    -1
+$EndComp
 Wire Wire Line
 	7050 1950 6950 1950
@@
 NoConn ~ 7050 2850
 $Comp
-L Switch:SW_Push_DPDT SW?
+L Switch:SW_Push_DPDT SW1
 U 1 1 5F1DCF29
 P 4850 2450
-F 0 "SW?" H 4650 2450 50  0000 C CNN
+F 0 "SW1" H 4650 2450 50  0000 C CNN
 F 1 "SW_Push_DPDT" H 4850 2016 50  0001 C CNN
-F 2 "" H 4850 2650 50  0001 C CNN
+F 2 "Button_Switch_THT:SW_NKK_GW12LJP" H 4850 2650 50  0001 C CNN
 F 3 "~" H 4850 2650 50  0001 C CNN
 	1    4850 2450
@@
 NoConn ~ 4650 2550
 NoConn ~ 4650 2750
-Wire Wire Line
-	2700 1750 2700 1900
-Text GLabel 2700 1850 2    50   Input ~ 0
+Text GLabel 3350 1350 2    50   Input ~ 0
 5V
 Text GLabel 6950 2000 0    50   Input ~ 0
@@
 5V
 $Comp
-L Device:C C?
+L Device:C C2
 U 1 1 5F1F55BF
 P 1900 5700
-F 0 "C?" H 1850 5450 50  0000 R CNN
+F 0 "C2" H 1850 5450 50  0000 R CNN
 F 1 "0.01uF" H 1850 5550 50  0000 R CNN
 F 2 "" H 1938 5550 50  0001 C CNN
@@
 $EndComp
 $Comp
-L power:GND #PWR?
+L power:GND #PWR0104
 U 1 1 5F1F65EE
 P 1900 5850
-F 0 "#PWR?" H 1900 5600 50  0001 C CNN
+F 0 "#PWR0104" H 1900 5600 50  0001 C CNN
 F 1 "GND" H 1905 5677 50  0000 C CNN
 F 2 "" H 1900 5850 50  0001 C CNN
@@
 	1900 5450 1900 5550
 $Comp
-L Device:C C?
+L Device:C C1
 U 1 1 5F1FA2F8
 P 1500 5700
-F 0 "C?" H 1400 5450 50  0000 R CNN
+F 0 "C1" H 1400 5450 50  0000 R CNN
 F 1 "1uF" H 1400 5550 50  0000 R CNN
 F 2 "" H 1538 5550 50  0001 C CNN
@@
 $EndComp
 $Comp
-L power:GND #PWR?
+L power:GND #PWR0105
 U 1 1 5F1FA741
 P 1500 5850
-F 0 "#PWR?" H 1500 5600 50  0001 C CNN
+F 0 "#PWR0105" H 1500 5600 50  0001 C CNN
 F 1 "GND" H 1505 5677 50  0000 C CNN
 F 2 "" H 1500 5850 50  0001 C CNN
@@
 	3150 5650 3200 5650
 $Comp
-L Device:R_POT RV?
+L Device:R_POT RV2
 U 1 1 5F1FB82A
 P 3600 5000
-F 0 "RV?" H 3850 5200 50  0000 R CNN
+F 0 "RV2" H 3850 5200 50  0000 R CNN
 F 1 "50K" H 3850 5100 50  0000 R CNN
-F 2 "" H 3600 5000 50  0001 C CNN
+F 2 "Connector_PinHeader_2.54mm:PinHeader_1x03_P2.54mm_Vertical" H 3600 5000 50  0001 C CNN
 F 3 "~" H 3600 5000 50  0001 C CNN
 	1    3600 5000
@@
 $EndComp
 $Comp
-L Device:R R?
+L Device:R R1
 U 1 1 5F1FDF15
 P 1500 5050
-F 0 "R?" H 1431 5004 50  0000 R CNN
+F 0 "R1" H 1431 5004 50  0000 R CNN
 F 1 "470K" H 1431 5095 50  0000 R CNN
-F 2 "" V 1430 5050 50  0001 C CNN
+F 2 "Resistor_THT:R_Axial_DIN0207_L6.3mm_D2.5mm_P2.54mm_Vertical" V 1430 5050 50  0001 C CNN
 F 3 "~" H 1500 5050 50  0001 C CNN
 	1    1500 5050
@@
 NoConn ~ 3150 5450
 $Comp
-L power:GND #PWR?
+L power:GND #PWR0106
 U 1 1 5F24F333
 P 2650 5850
-F 0 "#PWR?" H 2650 5600 50  0001 C CNN
+F 0 "#PWR0106" H 2650 5600 50  0001 C CNN
 F 1 "GND" H 2655 5677 50  0000 C CNN
 F 2 "" H 2650 5850 50  0001 C CNN
@@
 	1500 5250 1500 5550
 Wire Notes Line
-	4400 6300 1000 6300
+	5050 6300 1000 6300
 Wire Notes Line
-	1000 6300 1000 4300
+	1000 6300 1000 4100
 Wire Notes Line
-	1000 4300 4400 4300
+	1000 4100 5050 4100
 Wire Notes Line
-	4400 4300 4400 6300
-Text Notes 3950 6200 0    50   ~ 10
+	5050 4100 5050 6300
+Text Notes 4600 6200 0    50   ~ 10
 Oscillator
 Text GLabel 3850 5250 2    50   Input ~ 0
@@
 	3600 4800 3550 4800
 $Comp
-L Device:R R?
+L Device:R R2
 U 1 1 5F1FC01A
 P 3400 4800
-F 0 "R?" V 3193 4800 50  0000 C CNN
+F 0 "R2" V 3193 4800 50  0000 C CNN
 F 1 "330" V 3284 4800 50  0000 C CNN
-F 2 "" V 3330 4800 50  0001 C CNN
+F 2 "Resistor_THT:R_Axial_DIN0207_L6.3mm_D2.5mm_P2.54mm_Vertical" V 3330 4800 50  0001 C CNN
 F 3 "~" H 3400 4800 50  0001 C CNN
 	1    3400 4800
@@
 EN
 $Comp
-L Switch:SW_Push_DPDT SW?
+L Switch:SW_Push_DPDT SW2
 U 1 1 5F2920CA
 P 4850 3250
-F 0 "SW?" H 4650 3250 50  0000 C CNN
+F 0 "SW2" H 4650 3250 50  0000 C CNN
 F 1 "SW_Push_DPDT" H 4850 2816 50  0001 C CNN
-F 2 "" H 4850 3450 50  0001 C CNN
+F 2 "Button_Switch_THT:SW_NKK_GW12LJP" H 4850 3450 50  0001 C CNN
 F 3 "~" H 4850 3450 50  0001 C CNN
 	1    4850 3250
@@
 EN
 $Comp
-L power:GND #PWR?
+L power:GND #PWR0107
 U 1 1 5F1C5BB0
 P 4500 2400
-F 0 "#PWR?" H 4500 2150 50  0001 C CNN
+F 0 "#PWR0107" H 4500 2150 50  0001 C CNN
 F 1 "GND" H 4505 2227 50  0000 C CNN
 F 2 "" H 4500 2400 50  0001 C CNN
@@
 	4500 2350 4650 2350
 $Comp
-L power:GND #PWR?
+L power:GND #PWR0108
 U 1 1 5F2920C0
 P 4500 3200
-F 0 "#PWR?" H 4500 2950 50  0001 C CNN
+F 0 "#PWR0108" H 4500 2950 50  0001 C CNN
 F 1 "GND" H 4505 3027 50  0000 C CNN
 F 2 "" H 4500 3200 50  0001 C CNN
@@
 	4500 3150 4650 3150
 $Comp
-L Timer:NE555P U?
+L Timer:NE555P U1
 U 1 1 5F2154E9
 P 2650 5450
-F 0 "U?" H 2850 5950 50  0000 C CNN
+F 0 "U1" H 2850 5950 50  0000 C CNN
 F 1 "NE555P" H 2950 5850 50  0000 C CNN
 F 2 "Package_DIP:DIP-8_W7.62mm" H 3300 5050 50  0001 C CNN
@@
 	1    0    0    -1
 $EndComp
+$Comp
+L Regulator_Linear:AMS1117-5.0 U?
+U 1 1 5F228A3F
+P 3050 1350
+F 0 "U?" H 3050 1592 50  0000 C CNN
+F 1 "AMS1117-5.0" H 3050 1501 50  0000 C CNN
+F 2 "Package_TO_SOT_SMD:SOT-223-3_TabPin2" H 3050 1550 50  0001 C CNN
+F 3 "http://www.advanced-monolithic.com/pdf/ds1117.pdf" H 3150 1100 50  0001 C CNN
+	1    3050 1350
+	1    0    0    -1
+$EndComp
+Wire Wire Line
+	2000 1350 2600 1350
+$Comp
+L Device:C C?
+U 1 1 5F22DC3C
+P 2600 1500
+F 0 "C?" H 2400 1450 50  0000 R CNN
+F 1 "0.1uF" H 2500 1550 50  0000 R CNN
+F 2 "" H 2638 1350 50  0001 C CNN
+F 3 "~" H 2600 1500 50  0001 C CNN
+	1    2600 1500
+	1    0    0    1
+$EndComp
+Connection ~ 2600 1350
+Wire Wire Line
+	2600 1350 2750 1350
+$Comp
+L power:GND #PWR?
+U 1 1 5F22E669
+P 2600 1650
+F 0 "#PWR?" H 2600 1400 50  0001 C CNN
+F 1 "GND" H 2605 1477 50  0000 C CNN
+F 2 "" H 2600 1650 50  0001 C CNN
+F 3 "" H 2600 1650 50  0001 C CNN
+	1    2600 1650
+	1    0    0    -1
+$EndComp
+$Comp
+L Device:C C?
+U 1 1 5F231248
+P 4550 5200
+F 0 "C?" H 4350 5150 50  0000 R CNN
+F 1 "0.1uF" H 4450 5250 50  0000 R CNN
+F 2 "" H 4588 5050 50  0001 C CNN
+F 3 "~" H 4550 5200 50  0001 C CNN
+	1    4550 5200
+	-1   0    0    -1
+$EndComp
+Text GLabel 4550 5050 1    50   Input ~ 0
+5V
+$Comp
+L power:GND #PWR?
+U 1 1 5F231EDB
+P 4550 5350
+F 0 "#PWR?" H 4550 5100 50  0001 C CNN
+F 1 "GND" H 4555 5177 50  0000 C CNN
+F 2 "" H 4550 5350 50  0001 C CNN
+F 3 "" H 4550 5350 50  0001 C CNN
+	1    4550 5350
+	1    0    0    -1
+$EndComp

Commit message: NE555 schematic verified
Parts:
- C1, C2: footprint (none) -> Capacitor_THT:C_Disc_D4.3mm_W1.9mm_P5.00mm
- C3, C4: renamed from C?; footprint (none) -> Capacitor_SMD:C_0805_2012Metric_Pad1.15x1.40mm_HandSolder
- U1: footprint Package_DIP:DIP-8_W7.62mm -> Package_SO:SO-8_5.3x6.2mm_P1.27mm
- gave numbers to parts that had none: 1
Changed lines of the file:
@@
 F 0 "C2" H 1850 5450 50  0000 R CNN
 F 1 "0.01uF" H 1850 5550 50  0000 R CNN
-F 2 "" H 1938 5550 50  0001 C CNN
+F 2 "Capacitor_THT:C_Disc_D4.3mm_W1.9mm_P5.00mm" H 1938 5550 50  0001 C CNN
 F 3 "~" H 1900 5700 50  0001 C CNN
 	1    1900 5700
@@
 F 0 "C1" H 1400 5450 50  0000 R CNN
 F 1 "1uF" H 1400 5550 50  0000 R CNN
-F 2 "" H 1538 5550 50  0001 C CNN
+F 2 "Capacitor_THT:C_Disc_D4.3mm_W1.9mm_P5.00mm" H 1538 5550 50  0001 C CNN
 F 3 "~" H 1500 5700 50  0001 C CNN
 	1    1500 5700
@@
 F 0 "U1" H 2850 5950 50  0000 C CNN
 F 1 "NE555P" H 2950 5850 50  0000 C CNN
-F 2 "Package_DIP:DIP-8_W7.62mm" H 3300 5050 50  0001 C CNN
+F 2 "Package_SO:SO-8_5.3x6.2mm_P1.27mm" H 3300 5050 50  0001 C CNN
 F 3 "http://www.ti.com/lit/ds/symlink/ne555.pdf" H 3500 5050 50  0001 C CNN
 	1    2650 5450
@@
 $EndComp
 $Comp
-L Regulator_Linear:AMS1117-5.0 U?
+L Regulator_Linear:AMS1117-5.0 U2
 U 1 1 5F228A3F
 P 3050 1350
-F 0 "U?" H 3050 1592 50  0000 C CNN
+F 0 "U2" H 3050 1592 50  0000 C CNN
 F 1 "AMS1117-5.0" H 3050 1501 50  0000 C CNN
 F 2 "Package_TO_SOT_SMD:SOT-223-3_TabPin2" H 3050 1550 50  0001 C CNN
@@
 	2000 1350 2600 1350
 $Comp
-L Device:C C?
+L Device:C C3
 U 1 1 5F22DC3C
 P 2600 1500
-F 0 "C?" H 2400 1450 50  0000 R CNN
+F 0 "C3" H 2400 1450 50  0000 R CNN
 F 1 "0.1uF" H 2500 1550 50  0000 R CNN
-F 2 "" H 2638 1350 50  0001 C CNN
+F 2 "Capacitor_SMD:C_0805_2012Metric_Pad1.15x1.40mm_HandSolder" H 2638 1350 50  0001 C CNN
 F 3 "~" H 2600 1500 50  0001 C CNN
 	1    2600 1500
@@
 	2600 1350 2750 1350
 $Comp
-L power:GND #PWR?
+L power:GND #PWR0109
 U 1 1 5F22E669
 P 2600 1650
-F 0 "#PWR?" H 2600 1400 50  0001 C CNN
+F 0 "#PWR0109" H 2600 1400 50  0001 C CNN
 F 1 "GND" H 2605 1477 50  0000 C CNN
 F 2 "" H 2600 1650 50  0001 C CNN
@@
 $EndComp
 $Comp
-L Device:C C?
+L Device:C C4
 U 1 1 5F231248
 P 4550 5200
-F 0 "C?" H 4350 5150 50  0000 R CNN
+F 0 "C4" H 4350 5150 50  0000 R CNN
 F 1 "0.1uF" H 4450 5250 50  0000 R CNN
-F 2 "" H 4588 5050 50  0001 C CNN
+F 2 "Capacitor_SMD:C_0805_2012Metric_Pad1.15x1.40mm_HandSolder" H 4588 5050 50  0001 C CNN
 F 3 "~" H 4550 5200 50  0001 C CNN
 	1    4550 5200
@@
 5V
 $Comp
-L power:GND #PWR?
+L power:GND #PWR0110
 U 1 1 5F231EDB
 P 4550 5350
-F 0 "#PWR?" H 4550 5100 50  0001 C CNN
+F 0 "#PWR0110" H 4550 5100 50  0001 C CNN
 F 1 "GND" H 4555 5177 50  0000 C CNN
 F 2 "" H 4550 5350 50  0001 C CNN

Commit message: All footprints associated
Parts:
- J1: footprint (none) -> TerminalBlock:TerminalBlock_bornier-2_P5.08mm
- J2: footprint Connector_PinHeader_2.54mm:PinHeader_1x04_P2.54mm_Vertical -> Connector_PinSocket_2.54mm:PinSocket_1x04_P2.54mm_Vertical
Changed lines of the file:
@@
 F 0 "J1" H 1757 1775 50  0000 C CNN
 F 1 "Barrel_Jack" H 1757 1684 50  0000 C CNN
-F 2 "" H 1750 1410 50  0001 C CNN
+F 2 "TerminalBlock:TerminalBlock_bornier-2_P5.08mm" H 1750 1410 50  0001 C CNN
 F 3 "~" H 1750 1410 50  0001 C CNN
 	1    1700 1450
@@
 F 0 "J2" H 8272 2328 50  0000 R CNN
 F 1 "Conn_01x04_Male" H 8272 2373 50  0001 R CNN
-F 2 "Connector_PinHeader_2.54mm:PinHeader_1x04_P2.54mm_Vertical" H 8300 2400 50  0001 C CNN
+F 2 "Connector_PinSocket_2.54mm:PinSocket_1x04_P2.54mm_Vertical" H 8300 2400 50  0001 C CNN
 F 3 "~" H 8300 2400 50  0001 C CNN
 	1    8300 2400

Commit message: WIP
Connections:
- net at A1.3 (A2): now also J2.4 (Pin_4); no longer J2.3 (Pin_3)
- net at A1.4 (A1): now also J2.3 (Pin_3); no longer J2.4 (Pin_4)
Changed lines of the file:
@@
 $EndComp
-Wire Wire Line
-	7850 2550 8050 2550
-Wire Wire Line
-	8050 2550 8050 2500
-Wire Wire Line
-	8050 2500 8100 2500
-Wire Wire Line
-	7850 2450 8050 2450
-Wire Wire Line
-	8050 2450 8050 2400
-Wire Wire Line
-	8050 2400 8100 2400
-Wire Wire Line
-	7850 2250 8050 2250
-Wire Wire Line
-	8050 2250 8050 2300
-Wire Wire Line
-	8050 2300 8100 2300
-Wire Wire Line
-	7850 2150 8050 2150
-Wire Wire Line
-	8050 2150 8050 2200
-Wire Wire Line
-	8050 2200 8100 2200
 Wire Wire Line
 	7450 1500 7450 1650
@@
 	1    0    0    -1
 $EndComp
+Wire Wire Line
+	7850 2550 8050 2550
+Wire Wire Line
+	8050 2500 8100 2500
+Wire Wire Line
+	8050 2550 8050 2500
+Wire Wire Line
+	8050 2400 8100 2400
+Wire Wire Line
+	8050 2450 8050 2400
+Wire Wire Line
+	7850 2450 8050 2450
+Wire Wire Line
+	7850 2150 7950 2150
+Wire Wire Line
+	7950 2150 7950 2300
+Wire Wire Line
+	7950 2300 8100 2300
+Wire Wire Line
+	7850 2250 8000 2250
+Wire Wire Line
+	8000 2250 8000 2200
+Wire Wire Line
+	8000 2200 8100 2200
 $EndSCHEMATC
