File: stepper-tester.sch (KiCad schematic (older format))
At the start: 17 parts, among them J1 Barrel_Jack, J2 Conn_01x04_Male, Q1 BC547, SW1 SW_Push_DPDT, SW2 SW_Push_DPDT, U1 NE555P, U2 AMS1117-5.0

Commit message: WIP
Parts:
- C3, C4: footprint Capacitor_SMD:C_0805_2012Metric_Pad1.15x1.40mm_HandSolder -> Capacitor_SMD:C_0805_2012Metric_Pad1.18x1.45mm_HandSolder
Changed lines of the file:
@@
 F 0 "C3" H 2400 1450 50  0000 R CNN
 F 1 "0.1uF" H 2500 1550 50  0000 R CNN
-F 2 "Capacitor_SMD:C_0805_2012Metric_Pad1.15x1.40mm_HandSolder" H 2638 1350 50  0001 C CNN
+F 2 "Capacitor_SMD:C_0805_2012Metric_Pad1.18x1.45mm_HandSolder" H 2638 1350 50  0001 C CNN
 F 3 "~" H 2600 1500 50  0001 C CNN
 	1    2600 1500
@@
 F 0 "C4" H 4350 5150 50  0000 R CNN
 F 1 "0.1uF" H 4450 5250 50  0000 R CNN
-F 2 "Capacitor_SMD:C_0805_2012Metric_Pad1.15x1.40mm_HandSolder" H 4588 5050 50  0001 C CNN
+F 2 "Capacitor_SMD:C_0805_2012Metric_Pad1.18x1.45mm_HandSolder" H 4588 5050 50  0001 C CNN
 F 3 "~" H 4550 5200 50  0001 C CNN
 	1    4550 5200

Commit message: WIP
Parts:
- R2: footprint Resistor_THT:R_Axial_DIN0207_L6.3mm_D2.5mm_P2.54mm_Vertical -> Resistor_THT:R_Axial_DIN0204_L3.6mm_D1.6mm_P7.62mm_Horizontal
Changed lines of the file:
@@
 F 0 "R2" V 1543 4450 50  0000 C CNN
 F 1 "330" V 1634 4450 50  0000 C CNN
-F 2 "Resistor_THT:R_Axial_DIN0207_L6.3mm_D2.5mm_P2.54mm_Vertical" V 1680 4450 50  0001 C CNN
+F 2 "Resistor_THT:R_Axial_DIN0204_L3.6mm_D1.6mm_P7.62mm_Horizontal" V 1680 4450 50  0001 C CNN
 F 3 "~" H 1750 4450 50  0001 C CNN
 	1    1750 4450
