File: stepper-tester.kicad_pcb (KiCad board)
At the start: 2 copper layers, 81.3 x 40.6 mm, 18 parts, among them J1 Barrel_Jack, J2 Conn_01x04_Male, SW1 SW_Push_DPDT, SW2 SW_Push_DPDT, U1 NE555P, U2 AMS1117-5.0

Commit message: PCB
Parts:
- moved C1 9.35 mm to (119.5, 71.1)
- moved C4 1.49 mm to (135.1, 69.8), turned to 180 degrees
- moved C2 0.63 mm to (139.1, 72.7)
- moved R1 0.51 mm to (124.5, 75.2)
Routing:
- net 5V: track 0.00 -> 96.3 mm
- net VMOT: track 0.00 -> 68.1 mm
- net STEP: track 0.00 -> 29.3 mm
- net EN: track 0.00 -> 24.3 mm
- net Net-(C1-Pad2): track 0.00 -> 23.3 mm
- net DIR: track 0.00 -> 7.66 mm
- net GND: track 0.00 -> 6.35 mm, vias 0 -> 4
- net Net-(A1-Pad6): track 0.00 -> 5.08 mm
- net Net-(A1-Pad5): track 0.00 -> 5.08 mm
- net Net-(A1-Pad4): track 0.00 -> 5.08 mm
- net Net-(A1-Pad3): track 0.00 -> 5.08 mm
- net Net-(R2-Pad1): track 0.00 -> 4.06 mm
- net Net-(C2-Pad2): track 0.00 -> 2.99 mm
- added copper zone on F.Cu, net GND
Other:
- net class Default: clearance 0.2 -> 0.4; trace_width 0.25 -> 0.4
- net class POWER added: clearance 0.4, trace_width 1, via_dia 0.8, via_drill 0.4
- rule trace_clearance: 0.2 -> 0.4

Commit message: PCB cleanup
Parts:
- J1: value Barrel_Jack -> POWER
- SW1: value SW_Push_DPDT -> DIR SWITCH
- SW2: value SW_Push_DPDT -> ENABLE SWITCH
Routing:
- net GND: track 6.35 -> 11.4 mm

Commit message: new layout
Parts:
- moved C2 0.63 mm to (139.7, 72.7)
Routing:
- net GND: track 11.4 -> 209.3 mm
- net Net-(C2-Pad2): track 2.99 -> 3.63 mm
- removed copper zone on F.Cu, net GND
Other:
- net class Default: clearance 0.4 -> 0.3
- net class POWER: clearance 0.4 -> 0.3
- rule trace_clearance: 0.4 -> 0.3

Commit message: PCB WIP
Parts:
- added D1: 1N5817, Diode_THT:D_DO-41_SOD81_P10.16mm_Horizontal, F.Cu at (127.0, 81.3)
- added D2: 1N5817, Diode_THT:D_DO-41_SOD81_P10.16mm_Horizontal, F.Cu at (127.0, 86.4)
- added Q1: BC547, Package_TO_SOT_THT:TO-92L_Inline_Wide, F.Cu at (127.0, 76.2)
- A1, C1, C2, J2, R2, RV2: moved to F.Cu
- J1: value POWER -> Barrel_Jack; moved to F.Cu
- R1: value 470K -> 1K; moved to F.Cu
- SW1: value DIR SWITCH -> SW_Push_DPDT; moved to F.Cu
- SW2: value ENABLE SWITCH -> SW_Push_DPDT; moved to F.Cu
- moved SW1 34.2 mm to (96.5, 61.0), turned to 270 degrees
- moved A1 33.2 mm to (76.2, 61.0)
- moved C4 29.7 mm to (106.7, 78.5), turned to 90 degrees
- moved C2 27.6 mm to (114.4, 83.8), turned to 0 degrees
- moved J1 23.0 mm to (109.2, 55.9)
- moved R2 23.0 mm to (116.8, 66.0), turned to 180 degrees
- moved J2 21.3 mm to (71.1, 73.7)
- moved RV2 17.5 mm to (121.9, 66.0), turned to 0 degrees
- moved U1 15.8 mm to (116.8, 77.5)
- moved SW2 12.7 mm to (96.5, 73.7), turned to 270 degrees
- moved C3 12.0 mm to (128.5, 53.3), turned to 180 degrees
- moved C1 10.2 mm to (109.3, 71.1)
- moved R1 7.69 mm to (132.1, 76.2), turned to 90 degrees
- moved U2 3.92 mm to (128.3, 59.0), turned to 270 degrees
Connections:
- R1 pad 1: Net-(C1-Pad2) -> 5V
- R1 pad 2: 5V -> Net-(D2-Pad2)
- RV2 pad 2: STEP -> Net-(D1-Pad2)
- RV2 pad 3: STEP -> Net-(D1-Pad2)
Routing:
- net GND: track 209.3 -> 0.00 mm, vias 4 -> 0
- net 5V: track 96.3 -> 0.00 mm
- net VMOT: track 68.1 -> 0.00 mm
- net STEP: track 29.3 -> 0.00 mm
- net EN: track 24.3 -> 0.00 mm
- net Net-(C1-Pad2): track 23.3 -> 0.00 mm
- net DIR: track 7.66 -> 0.00 mm
- net Net-(A1-Pad6): track 5.08 -> 0.00 mm
- net Net-(A1-Pad5): track 5.08 -> 0.00 mm
- net Net-(A1-Pad4): track 5.08 -> 0.00 mm
- net Net-(A1-Pad3): track 5.08 -> 0.00 mm
- net Net-(R2-Pad1): track 4.06 -> 0.00 mm
- net Net-(C2-Pad2): track 3.63 -> 0.00 mm

Commit message: WIP
Parts:
- removed REF** (x4): MountingHole_3.2mm_M3_DIN965_Pad, MountingHole:MountingHole_3.2mm_M3_DIN965_Pad
- C3, C4: moved to B.Cu
- moved J1 27.9 mm to (81.3, 55.9)
- moved C3 8.96 mm to (133.2, 61.0)
- moved C1 8.81 mm to (118.1, 71.0), turned to 90 degrees
- moved U2 6.73 mm to (131.9, 64.7)
- moved R2 5.68 mm to (121.9, 63.5)
- moved D2 5.08 mm to (127.0, 81.3)
- moved SW2 3.59 mm to (99.1, 76.2)
- moved SW1 3.59 mm to (99.1, 63.5)
- moved C2 3.54 mm to (116.8, 86.4)
- moved U1 2.65 mm to (115.6, 79.8)
- moved C4 2.64 mm to (108.0, 76.2), turned to 0 degrees
- moved D1 2.54 mm to (127.0, 78.7)
- moved J2 2.54 mm to (71.1, 76.2)
- moved A1 2.54 mm to (76.2, 63.5)
Routing:
- net 5V: track 0.00 -> 34.1 mm, vias 0 -> 5
- net GND: track 0.00 -> 14.5 mm, vias 0 -> 3
- net Net-(D1-Pad1): track 0.00 -> 10.6 mm, vias 0 -> 1
- net Net-(C1-Pad2): track 0.00 -> 9.29 mm, vias 0 -> 2
- net VMOT: track 0.00 -> 8.32 mm, vias 0 -> 1
- net Net-(D1-Pad2): track 0.00 -> 7.62 mm
- net Net-(C2-Pad2): track 0.00 -> 6.25 mm, vias 0 -> 1
- net Net-(D2-Pad2): track 0.00 -> 5.08 mm
- net Net-(A1-Pad6): track 0.00 -> 5.08 mm
- net Net-(A1-Pad5): track 0.00 -> 5.08 mm
- net Net-(A1-Pad4): track 0.00 -> 5.08 mm
- net Net-(A1-Pad3): track 0.00 -> 5.08 mm
- net STEP: track 0.00 -> 3.24 mm, vias 0 -> 1
- net Net-(R2-Pad1): track 0.00 -> 2.54 mm

Commit message: WIP
Parts:
- C3, C4: footprint Capacitor_SMD:C_0805_2012Metric_Pad1.15x1.40mm_HandSolder -> Capacitor_SMD:C_0805_2012Metric_Pad1.18x1.45mm_HandSolder
- R2: footprint Resistor_THT:R_Axial_DIN0207_L6.3mm_D2.5mm_P2.54mm_Vertical -> Resistor_THT:R_Axial_DIN0204_L3.6mm_D1.6mm_P7.62mm_Horizontal
- moved C3 28.4 mm to (105.2, 55.9)
- moved U2 28.4 mm to (104.0, 59.6)
- moved C1 11.7 mm to (109.2, 63.5)
- moved R1 11.4 mm to (121.9, 71.1)
- moved D1 11.4 mm to (116.8, 73.7)
- moved D2 11.4 mm to (116.8, 76.2)
- moved Q1 11.4 mm to (116.8, 71.1)
- moved C2 9.16 mm to (109.2, 81.3)
- moved RV2 9.16 mm to (116.8, 58.4)
- moved U1 9.16 mm to (108.0, 74.7)
- moved C4 9.16 mm to (100.3, 71.1)
- moved R2 9.16 mm to (116.8, 55.9)
- moved SW2 3.59 mm to (96.5, 78.7)
- moved SW1 2.54 mm to (96.5, 63.5)
Routing:
- net DIR: track 0.00 -> 7.62 mm
- net EN: track 0.00 -> 5.08 mm
- net 5V: track 34.1 -> 36.9 mm
- net Net-(D1-Pad2): track 7.62 -> 5.08 mm
- net Net-(D1-Pad1): track 10.6 -> 8.07 mm
Other:
- board size 81.3 x 40.6 mm -> 61 x 40.6 mm

Commit message: Add readme
Parts:
- SW1: value SW_Push_DPDT -> DIR
- SW2: value SW_Push_DPDT -> EN
Changed lines of the file:
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@@
       (effects (font (size 1 1) (thickness 0.15)))
     )
-    (fp_text value 1uF (at 2.5 2.2 90) (layer F.Fab)
+    (fp_text value 1uF (at 2.5 2.2 90) (layer F.Fab) hide
       (effects (font (size 1 1) (thickness 0.15)))
     )
@@
       (effects (font (size 1 1) (thickness 0.15)))
     )
-    (fp_text value Barrel_Jack (at 2.54 5.08) (layer F.Fab)
+    (fp_text value Barrel_Jack (at -7.62 2.54) (layer F.Fab) hide
       (effects (font (size 1 1) (thickness 0.15)))
     )
@@
     (fp_line (start -2.46 -3.75) (end -2.46 3.75) (layer F.Fab) (width 0.1))
     (fp_line (start -2.41 2.55) (end 7.49 2.55) (layer F.Fab) (width 0.1))
-    (fp_text user %R (at 2.54 0) (layer F.Fab)
+    (fp_text user %R (at 8.89 1.27) (layer F.Fab)
       (effects (font (size 1 1) (thickness 0.15)))
     )
@@
       (effects (font (size 1 1) (thickness 0.15)))
     )
-    (fp_text value BC547 (at 2.54 2.79 90) (layer F.Fab)
+    (fp_text value BC547 (at 2.54 2.79 90) (layer F.Fab) hide
       (effects (font (size 1 1) (thickness 0.15)))
     )
@@
       (effects (font (size 1 1) (thickness 0.15)))
     )
-    (fp_text value 1K (at 1.27 2.37 90) (layer F.Fab)
+    (fp_text value 1K (at 1.27 2.37 90) (layer F.Fab) hide
       (effects (font (size 1 1) (thickness 0.15)))
     )
@@
       (effects (font (size 1 1) (thickness 0.15)))
     )
-    (fp_text value 50K (at 0 7.41) (layer F.Fab)
+    (fp_text value 50K (at 3.81 2.54) (layer F.Fab) hide
       (effects (font (size 1 1) (thickness 0.15)))
     )
@@
     (fp_line (start 1.27 -1.27) (end 1.27 6.35) (layer F.Fab) (width 0.1))
     (fp_line (start -0.635 -1.27) (end 1.27 -1.27) (layer F.Fab) (width 0.1))
-    (fp_text user %R (at 0 2.54 90) (layer F.Fab)
+    (fp_text user %R (at 3.81 2.54 180) (layer F.Fab)
       (effects (font (size 1 1) (thickness 0.15)))
     )
@@
       (effects (font (size 1 1) (thickness 0.15)))
     )
-    (fp_text value SW_Push_DPDT (at 2.54 4.52 90) (layer F.Fab)
+    (fp_text value DIR (at -2.54 1.27 180) (layer F.Fab)
       (effects (font (size 1 1) (thickness 0.15)))
     )
@@
       (effects (font (size 1 1) (thickness 0.15)))
     )
-    (fp_text value SW_Push_DPDT (at 2.54 4.52 90) (layer F.Fab)
+    (fp_text value EN (at -2.54 1.27 180) (layer F.Fab)
       (effects (font (size 1 1) (thickness 0.15)))
     )
@@
       (effects (font (size 1 1) (thickness 0.15)))
     )
-    (fp_text value AMS1117-5.0 (at 0 4.5 90) (layer F.Fab)
+    (fp_text value AMS1117-5.0 (at -7.52788 -0.143433 180) (layer F.Fab)
       (effects (font (size 1 1) (thickness 0.15)))
     )
@@
       (effects (font (size 1 1) (thickness 0.15)))
     )
-    (fp_text value 330 (at 3.81 1.92) (layer F.Fab)
-      (effects (font (size 1 1) (thickness 0.15)))
-    )
+    (fp_text value 330 (at 3.81 1.92) (layer F.Fab) hide
+      (effects (font (size 1 1) (thickness 0.15)))
+    )
